File: aek2_usb_Teensy.kicad_pcb (KiCad board)
At the start: 2 copper layers, 439 x 141.6 mm, 241 parts, among them J1 Conn_01x04, J2 Conn_01x04, U1 ATmega32A-PU

Commit message: Committed initial kicad files for modified PCB
Parts:
- removed AVR1: AVR-ISP-6, Connector_PinHeader_2.54mm:PinHeader_2x03_P2.54mm_Horizontal
- removed Boot1: Boot, Button_Switch_THT:SW_PUSH_6mm
- removed C1: 4.7u, Capacitor_THT:CP_Radial_D5.0mm_P2.50mm
- removed C2, C3: 0.1u, Capacitor_THT:C_Disc_D3.0mm_W2.0mm_P2.50mm
- removed C4, C5: 22p, Capacitor_THT:C_Disc_D6.0mm_W2.5mm_P5.00mm
- removed D1, D2: 3.6V, Diode_THT:D_DO-35_SOD27_P7.62mm_Horizontal
- removed F1: 500mA, Fuse:Fuse_Littelfuse_395Series
- removed R1: 1.5K, Resistor_THT:R_Axial_DIN0207_L6.3mm_D2.5mm_P10.16mm_Horizontal
- removed R2, R3: 68R, Resistor_THT:R_Axial_DIN0207_L6.3mm_D2.5mm_P10.16mm_Horizontal
- removed R4: 10k, Resistor_THT:R_Axial_DIN0207_L6.3mm_D2.5mm_P10.16mm_Horizontal
- removed Reset1: Reset, Button_Switch_THT:SW_PUSH_6mm
- removed XTAL1: Crystal, Crystal:Crystal_HC49-4H_Vertical
- added J3: Conn_01x04, Connector_JST:JST_PH_S4B-PH-K_1x04_P2.00mm_Horizontal, F.Cu at (268.0, 151.9)
- U1: value ATmega32A-PU -> Teensy++ 2.0
- moved G*** 4.86 mm to (386.1, 148.6)
- moved G*** 1.27 mm to (188.0, 147.8)
Connections:
- U1 pad 10: +5V -> (no net)
- U1 pad 18: boot -> col12
- U1 pad 20: col12 -> GND
- U1 pad 30: +5V -> (no net)
Routing:
- net +5V: track 449.6 -> 0.00 mm
- net reset: track 183.0 -> 0.00 mm
- net MISO: track 166.1 -> 0.00 mm
- net MOSI: track 166.0 -> 0.00 mm
- net SCK: track 166.0 -> 0.00 mm
- net boot: track 156.6 -> 0.00 mm
- net D+: track 60.6 -> 0.00 mm
- net D-: track 54.7 -> 0.00 mm
- net Net-(C5-Pad1): track 49.8 -> 0.00 mm
- net Net-(C4-Pad1): track 48.9 -> 0.00 mm
- net JST-D-: track 495.9 -> 464.2 mm, vias 0 -> 2
- net JST-D+: track 482.5 -> 459.8 mm
- net col12: track 256.7 -> 261.1 mm, vias 0 -> 2
- net VCC: track 467.6 -> 464.0 mm
- added copper zone on B.Cu, net boot
Other:
- board text added: "+LL"
- board text added: "AEK II USB Teensy PCB rev. 1"
- board text added: "github.com/linuxleah/teensy_aek2_usb forked from aek2_usb by kb-elmo"
- board text removed: "AEK II USB PCB rev. 1"
- board text removed: "MOSI"
- board text removed: "RST"
- board text removed: "github.com/kb-elmo/aek2_usb elmo.space"
