File: aek2_usb_Teensy.sch (KiCad schematic (older format))
At the start: 237 parts, among them J1 Conn_01x04, J2 Conn_01x04, U1 ATmega32A-PU

Commit message: Committed initial kicad files for modified PCB
Parts:
- removed AVR1: AVR-ISP-6, Connector_PinHeader_2.54mm:PinHeader_2x03_P2.54mm_Horizontal, symbol Connector:AVR-ISP-6
- removed Boot1: Boot, Button_Switch_THT:SW_PUSH_6mm, symbol Switch:SW_Push
- removed C1: 4.7u, Capacitor_THT:CP_Radial_D5.0mm_P2.50mm, symbol Device:CP1
- removed C2, C3: 0.1u, Capacitor_THT:C_Disc_D3.0mm_W2.0mm_P2.50mm, symbol Device:C
- removed C4, C5: 22p, Capacitor_THT:C_Disc_D6.0mm_W2.5mm_P5.00mm, symbol Device:C_Small
- removed D1, D2: 3.6V, Diode_THT:D_DO-35_SOD27_P7.62mm_Horizontal, symbol Device:D_Zener
- removed F1: 500mA, Fuse:Fuse_Littelfuse_395Series, symbol Device:Polyfuse
- removed R1: 1.5K, Resistor_THT:R_Axial_DIN0207_L6.3mm_D2.5mm_P10.16mm_Horizontal, symbol Device:R
- removed R2, R3: 68R, Resistor_THT:R_Axial_DIN0207_L6.3mm_D2.5mm_P10.16mm_Horizontal, symbol Device:R
- removed R4: 10k, Resistor_THT:R_Axial_DIN0207_L6.3mm_D2.5mm_P10.16mm_Horizontal, symbol Device:R
- removed Reset1: Reset, Button_Switch_THT:SW_PUSH_6mm, symbol Switch:SW_Push
- removed XTAL1: Crystal, Crystal:Crystal_HC49-4H_Vertical, symbol Device:Crystal
- added J3: Conn_01x04, Connector_JST:JST_PH_S4B-PH-K_1x04_P2.00mm_Horizontal, symbol aek2_usb-rescue:Conn_01x04-Connector_Generic
- D10, D100, D101, D102, D103, D104, D105, D106, D107, D11, D12, D13, D14, D15, D16, D17, D18, D19, D20, D21, D22, D23, D24, D25, D26, D27, D28, D29, D3, D30, D31, D32, D33, D34, D35, D36, D37, D38, D39, D4, D40, D41, D42, D43, D44, D45, D46, D47, D48, D49, D5, D50, D51, D52, D53, D54, D55, D56, D57, D58, D59, D6, D60, D61, D62, D63, D64, D65, D66, D67, D68, D69, D7, D70, D71, D72, D73, D74, D75, D76, D77, D78, D79, D8, D80, D81, D82, D83, D84, D85, D86, D87, D88, D89, D9, D90, D91, D92, D93, D94, D95, D96, D97, D98, D99: symbol Device:D_Small -> aek2_usb-rescue:D_Small-Device
- H1, H2: symbol Mechanical:MountingHole_Pad -> aek2_usb-rescue:MountingHole_Pad-Mechanical
- J1, J2: symbol Connector_Generic:Conn_01x04 -> aek2_usb-rescue:Conn_01x04-Connector_Generic
- LED1, LED2, LED3: symbol Device:LED -> aek2_usb-rescue:LED-Device
- MX1, MX10, MX100, MX101, MX102, MX103, MX104, MX105, MX11, MX12, MX13, MX14, MX15, MX16, MX17, MX18, MX19, MX2, MX20, MX21, MX22, MX23, MX24, MX25, MX26, MX27, MX28, MX29, MX3, MX30, MX31, MX32, MX33, MX34, MX35, MX36, MX37, MX38, MX39, MX4, MX40, MX41, MX42, MX43, MX44, MX45, MX46, MX47, MX48, MX49, MX5, MX50, MX51, MX52, MX53, MX54, MX55, MX56, MX57, MX58, MX59, MX6, MX60, MX61, MX62, MX63, MX64, MX65, MX66, MX67, MX68, MX69, MX7, MX70, MX71, MX72, MX73, MX74, MX75, MX76, MX77, MX78, MX79, MX8, MX80, MX81, MX82, MX83, MX84, MX85, MX86, MX87, MX88, MX89, MX9, MX90, MX91, MX92, MX93, MX94, MX95, MX96, MX97, MX98, MX99: symbol MX_Alps_Hybrid:MX-NoLED -> aek2_usb-rescue:MX-NoLED-MX_Alps_Hybrid
- R5, R6, R7: symbol Device:R -> aek2_usb-rescue:R-Device
- U1: symbol MCU_Microchip_ATmega:ATmega32A-PU -> aek2_usb-rescue:ATmega32A-PU-MCU_Microchip_ATmega
Connections:
- net labels removed: +5V, reset
- wire segments 344 -> 300
